Commit message: Misc changes

File: meshes/ur3_joint_limited_robot_new.urdf (robot description, URDF)
Before this commit: robot ur3, 11 links, 10 joints
Links:
- link base_link: geometry collision mesh filename=collision/base.stl; visual mesh filename=visual/base.stl
- link forearm_link: geometry collision mesh filename=collision/forearm.stl; visual mesh filename=visual/forearm.stl
- link shoulder_link: geometry collision mesh filename=collision/shoulder.stl; visual mesh filename=visual/shoulder.stl
- link tool0: geometry collision mesh filename=collision/grounded_peg.stl scale=0.001 0.001 0.001; visual mesh filename=collision/grounded_peg.stl scale=0.001 0.001 0.001
- link upper_arm_link: geometry collision mesh filename=collision/upperarm.stl; visual mesh filename=visual/upperarm.stl
- link wrist_1_link: geometry collision mesh filename=collision/wrist1.stl; visual mesh filename=visual/wrist1.stl
- link wrist_2_link: geometry collision mesh filename=collision/wrist2.stl; visual mesh filename=visual/wrist2.stl
- link wrist_3_link: geometry collision mesh filename=collision/wrist3.stl; visual mesh filename=visual/wrist3.stl
Joints:
- joint world_joint: parent world -> ground_plane_box

File: urdf/ur3_joint_limited_robot_new.urdf (robot description, URDF)
Before this commit: robot ur3, 11 links, 10 joints
Links:
- link base_link: geometry collision mesh filename=package://impedance_test/meshes/collision/base.stl; visual mesh filename=package://impedance_test/meshes/visual/base.dae
- link forearm_link: geometry collision mesh filename=package://impedance_test/meshes/collision/forearm.stl; visual mesh filename=package://impedance_test/meshes/visual/forearm.dae
- link shoulder_link: geometry collision mesh filename=package://impedance_test/meshes/collision/shoulder.stl; visual mesh filename=package://impedance_test/meshes/visual/shoulder.dae
- link tool0: geometry collision mesh filename=package://impedance_test/meshes/collision/grounded_peg.stl scale=0.001 0.001 0.001; visual mesh filename=package://impedance_test/meshes/collision/grounded_peg.stl scale=0.001 0.001 0.001
- link upper_arm_link: geometry collision mesh filename=package://impedance_test/meshes/collision/upperarm.stl; visual mesh filename=package://impedance_test/meshes/visual/upperarm.dae
- link wrist_1_link: geometry collision mesh filename=package://impedance_test/meshes/collision/wrist1.stl; visual mesh filename=package://impedance_test/meshes/visual/wrist1.dae
- link wrist_2_link: geometry collision mesh filename=package://impedance_test/meshes/collision/wrist2.stl; visual mesh filename=package://impedance_test/meshes/visual/wrist2.dae
- link wrist_3_link: geometry collision mesh filename=package://impedance_test/meshes/collision/wrist3.stl; visual mesh filename=package://impedance_test/meshes/visual/wrist3.dae
